File: electronotes/misc/high-ripple-vcf-en90-11-lm13700s.sch (EAGLE design)
At the start: 111 parts, among them IC1 TL074, IC10 CA3080E, IC11 TL074, IC12 CA3080E, IC13 CA3080E, IC2 TL072, IC3 TL072, IC4 CA3080E, IC5 CA3080E, IC6 TL072, IC7 TL072, IC8 TL074, IC9 CA3080E, T1 3904, T2 3906, T3 3906, T4 3906, T5 3906, T6 3906, T7 3906

Commit message: Add new versions of the high ripple vcf and vocal filter
Parts:
- removed AN3, ENV3: (no value), wirepad:2,54/1,0
- removed IC10, IC12, IC13, IC9: CA3080E, mmoretti:CA3080E
- removed IC2, IC3, IC6, IC7: TL072, mmoretti:TL072-TOPP
- added ANIM, CVLVL, ENV: B100k, mmoretti:POT-ATTEN
- added C17, C18, C19, C20, C21, C22, C23, C24, C25, C26, C27, C28: .1uF, rcl:C-US025-025X050
- added GND: (no value), wirepad:2,15/1,0
- added IC14, IC15, IC16: LM13700N, mmoretti:LM13700N
- added IFRQ: B100k, mmoretti:POT
- AN1, AN2, CV, ENV2, IN, INI1, INI2, INI3, OUT: device wirepad:2,54/1,0 -> wirepad:2,15/1,0
- C1, C10, C11, C12, C2, C3, C4, C9: device rcl:C-US050-025X075 -> rcl:C-US025-025X050
- HFC: value 500 -> 500R
- IC4, IC5: value CA3080E -> TL074; device mmoretti:CA3080E -> mmoretti:TL074-TOPP
- R1, R10, R11, R12, R14, R15, R17, R19, R2, R21, R22, R23, R25, R27, R3, R30, R31, R32, R33, R35, R36, R37, R4, R40, R41, R42, R5, R6, R7, R8, R9, RA-A1, RA-A2, RA-A3, RA-B1, RA-B2, RA-B3, RT1, RT2, RT3: device rcl:R-US_0207/10 -> rcl:R-US_0207/2V
- R45: device rcl:R-US_0207/10 -> rcl:R-US_0207/5V
Connections:
- net +12V: now also C17.1, C19.1, C21.1, C23.1, C25.1, C27.1, IC14SUPPLY.7, IC15SUPPLY.7, IC16SUPPLY.7, IC4P.V+, IC5P.V+, IFRQ.1; no longer IC10G$2.7, IC12G$2.7, IC13G$2.7, IC2P.V+, IC3P.V+, IC4G$2.7, IC5G$2.7, IC6P.V+, IC7P.V+, IC9G$2.7
- net -12V: now also C18.2, C20.2, C22.2, C24.2, C26.2, C28.2, IC14SUPPLY.4, IC15SUPPLY.4, IC16SUPPLY.4, IC4P.V-, IC5P.V-, IFRQ.3; no longer IC10G$2.4, IC12G$2.4, IC13G$2.4, IC2P.V-, IC3P.V-, IC4G$2.4, IC5G$2.4, IC6P.V-, IC7P.V-, IC9G$2.4
- net A: now also IC15OTA1.I_BIAS; no longer IC4G$1.I_BIAS
- net B: now also IC15OTA2.I_BIAS; no longer IC5G$1.I_BIAS
- net C: now also IC14OTA1.I_BIAS; no longer IC9G$1.I_BIAS
- net D: now also IC14OTA2.I_BIAS; no longer IC10G$1.I_BIAS
- net E: now also IC16OTA1.I_BIAS; no longer IC12G$1.I_BIAS
- net GND: now also C27.2, C28.1, GND.P, IC14OTA1.IN_P, IC14OTA2.IN_P, IC15OTA1.IN_P, IC15OTA2.IN_P, IC16OTA1.IN_P, IC16OTA2.IN_P, IC4A.-IN, IC4B.+IN, IC4C.+IN, IC4D.-IN, IC5A.+IN, IC5B.+IN, IC5C.-IN, IC5D.+IN, RA-A3.2; no longer AN3.P, C1.2, C2.1, C3.2, C4.1, ENV3.P, IC10G$1.IN_P, IC12G$1.IN_P, IC13G$1.IN_P, IC2A.+IN, IC2B.+IN, IC3A.+IN, IC3B.-IN, IC4G$1.IN_P, IC5G$1.IN_P, IC6A.+IN, IC6B.-IN, IC7A.+IN, IC7B.-IN, IC9G$1.IN_P, RA-A3.1
- net N$1: now also IC5A.-IN; no longer IC2B.-IN
- net N$16: now also IC4C.OUT; no longer IC3A.OUT
- net N$17: now also IC4D.+IN; no longer IC3B.+IN
- net N$18: now also IC4D.OUT; no longer IC3B.OUT
- net N$2: now also CVLVL.2
- net N$20: now also IC4B.OUT; no longer IC6A.OUT
- net N$21: now also IC4C.-IN; no longer IC3A.-IN
- net N$22: now also IC4A.+IN; no longer IC6B.+IN
- net N$23: now also IC4A.OUT; no longer IC6B.OUT
- net N$25: now also IC4B.-IN; no longer IC6A.-IN
- net N$26: now also IC5D.OUT; no longer IC7A.OUT
- net N$27: now also IC5C.+IN; no longer IC7B.+IN
- net N$28: now also IC5C.OUT; no longer IC7B.OUT
- net N$3: now also IFRQ.2, R2.2; no longer R2.1
- net N$30: now also IC5D.-IN; no longer IC7A.-IN
- net N$31: now also IC11B.OUT; no longer IC1C.OUT
- net N$32: now also IC8C.OUT; no longer IC8B.OUT
- net N$34: now also IC14OTA1.IN_N; no longer IC9G$1.IN_N
- net N$35: now also IC14OTA1.OUT, IC8D.-IN; no longer IC8A.-IN, IC9G$1.OUT
- net N$36: now also IC11C.OUT; no longer IC1B.OUT
- net N$38: now also IC15OTA1.IN_N; no longer IC4G$1.IN_N
- net N$39: now also IC11D.-IN, IC15OTA1.OUT; no longer IC1A.-IN, IC4G$1.OUT
- net N$4: now also ENV.2
- net N$40: now also IC11D.OUT; no longer IC1A.OUT
- net N$41: now also IC8D.OUT; no longer IC8A.OUT
- net N$43: now also IC15OTA2.IN_N; no longer IC5G$1.IN_N
- net N$44: now also IC11B.-IN, IC15OTA2.OUT; no longer IC1C.-IN, IC5G$1.OUT
- net N$45: now also IC11C.-IN; no longer IC1B.-IN
- net N$46: now also IC11A.-IN, IC11A.OUT; no longer IC1D.-IN, IC1D.OUT
- net N$48: now also IC14OTA2.IN_N; no longer IC10G$1.IN_N
- net N$49: now also IC14OTA2.OUT, IC8B.-IN; no longer IC10G$1.OUT, IC8C.-IN
- net N$5: now also ANIM.2
- net N$50: now also IC8C.-IN; no longer IC8B.-IN
- net N$51: now also IC8A.-IN, IC8A.OUT; no longer IC8D.-IN, IC8D.OUT
- net N$52: now also IC8B.OUT; no longer IC8C.OUT
- net N$53: now also IC1C.OUT; no longer IC11B.OUT
- net N$55: now also IC16OTA1.IN_N, RA-A3.1; no longer IC12G$1.IN_N, RA-A3.2
- net N$56: now also IC16OTA1.OUT, IC1D.-IN; no longer IC11A.-IN, IC12G$1.OUT
- net N$57: now also IC1D.OUT; no longer IC11A.OUT
- net N$59: now also IC16OTA2.IN_N; no longer IC13G$1.IN_N
- net N$6: now also IC5B.-IN, R2.1; no longer IC2A.-IN, R2.2
- net N$60: now also IC16OTA2.OUT, IC1B.-IN; no longer IC11C.-IN, IC13G$1.OUT
- net N$61: now also IC1C.-IN; no longer IC11B.-IN
- net N$62: now also IC1A.-IN, IC1A.OUT; no longer IC11D.-IN, IC11D.OUT
- net N$63: now also IC1B.OUT; no longer IC11C.OUT
- net N$66: now also IC16OTA2.I_BIAS; no longer IC13G$1.I_BIAS
- net N$8: now also IC5B.OUT; no longer IC2A.OUT
- net X: now also ANIM.1, IC5A.OUT; no longer IC2B.OUT
Other:
- note added: "pin1 to CV input"
- note added: "pin1 to ENV input"
- note removed: "100k pot"
- note removed: "100k pot pin1 to ENV input"
- moved on the sheet: C1, C2, C5, C6, IC11A, IC11B, IC11C, IC11D, IC1A, IC1B, IC1C, IC1D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
