File: electronotes/ens-76/en76-vco4.sch (EAGLE design)
At the start: 112 parts, among them IC1 TL072P, IC2 TL074, IC3 TL074, IC4 LM13700, IC5 TL072P, IC6 CA3080E, IC7 4066N, IC8 4066N, IC9 CA3080E, T1 3906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

Commit message: Add pot symbols to make things clearer
Parts:
- added COARSE, FINE, INIFRQ: (no value), mmoretti:POT
- added CVLVL, ENVLVL, EXTMOD, INIDPTH, SELFMOD: (no value), mmoretti:POT-ATTEN
Connections:
- net +12V: now also COARSE.1, FINE.1, INIDPTH.1, INIFRQ.1
- net -12V: now also COARSE.3, FINE.3, INIFRQ.3
- net N$1: now also COARSE.2
- net N$12: now also FINE.2
- net N$2: now also CVLVL.2
- net N$27: now also INIFRQ.2
- net N$48: now also INIDPTH.2
- net N$50: now also ENVLVL.2
- net N$51: now also EXTMOD.2
- net N$52: now also SELFMOD.2
Other:
- note added: "To CV jack"
- note added: "To jack"
- note removed: "CV1 (pot pin) to CV jack CV3 (pot pin) to GNDP"
- note removed: "ID3 pot pin to GNDP ENV1 pot pin to jack ENV3 pot pin to GNDP"
- note removed: "SM3 pot pin to GNDP EM1 pot pin to jack EM3 pot pin to GNDP"
- moved on the sheet: 1VO, CT1, CT2, CT3, CV2, D9, EM2, ENV2, FT1, FT2, FT3, IC5A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
